File: lil-flite/Connectors.kicad_sch (KiCad schematic)
At the start: 14 parts, among them J101 USB4105-GF-A, J202 Conn_01x02, J203 Conn_01x02, J204 Conn_02x06_Odd_Even, T201 AO3401A

Commit message: Almost finished
Need to double check everything
routing done
more vias maybe
Parts:
- added D202: 1N4148W-7-F, SOD3716X145N, symbol SamacSys_Parts:1N4148W-7-F
- added R401: 330R, Resistor_SMD:R_0603_1608Metric_Pad0.98x0.95mm_HandSolder, symbol PCM_Generic-50:R,IEC
- added R406 (x2): 5k1, Resistor_SMD:R_0603_1608Metric_Pad0.98x0.95mm_HandSolder, symbol PCM_Generic-50:R,IEC
- added R406 (x2): 10k, Resistor_SMD:R_0603_1608Metric_Pad0.98x0.95mm_HandSolder, symbol PCM_Generic-50:R,IEC
- added R406: 1k, Resistor_SMD:R_0603_1608Metric_Pad0.98x0.95mm_HandSolder, symbol PCM_Generic-50:R,IEC
- added T202, T203: AO3401A, JLC-Transistors:SOT23-3L, symbol JLC-Transistors:AO3401A
- BZ201: value Buzzer -> CMT-8504-100-SMT-TR; footprint lil-flite:CMT-8504-100-SMT-TR -> lil-flite:XDCR_CMT-8504-100-SMT-TR
Connections:
- net +5V: now also D202.2 (A), R406.1 (+), T202.1
- net +BATT: now also T202.3, T203.2; no longer C407.2 (-), PS101.3 (VIN)
- net GND: now also BZ201.N (+), D101.2 (A), R406.1 (+), R406.1 (+), R406.1 (+), R406.1 (+), R406.2 (-); no longer BZ201.2 (+)
- net RECOVERY_LED: now also T203.3
- net USB.CC1: now also R406.2 (-)
- net USB.CC2: now also R406.2 (-)
- net VCC: now also R401.2 (-)
- net at T201.3: now also BZ201.P (-); no longer BZ201.1 (-)
- net at D101.1 (K): now also R401.1 (+)
- net MISC.Buzzer_PWM: now reaches T201.1
- net MISC.Buzzer_PWM: now also R406.2 (-)
- new net: C407.2 (-), D202.1 (K), PS101.3 (VIN), T202.2
- new net MISC.RECOVERY_LED_PWM: R406.2 (-), T203.1
Other:
- moved on the sheet: BZ201, D101, T201
