File: lil-flite/lil-flite.kicad_sch (KiCad schematic)
At the start: 0 parts

Commit message: Almost finished
Need to double check everything
routing done
more vias maybe
Other:
- sheet Connectors + Power ports: added JTAG{DOSWO,NJTRST,MSSWDIO,CLK,DI}, MISC{RECOVERY_LED_PWM,Buzzer_PWM}, USB{Data_-,Data_+,CC1,CC2}; removed JTAG{DO&SWO,NJTRST,MS&SWDIO,CLK,DI}
- sheet MCU ports: added BMP{MOSI,MISO,SCK,NSS}, IMU{SCL,SDA,INTA,INTM}, JTAG{DOSWO,NJTRST,MSSWDIO,CLK,DI}, MISC{RECOVERY_LED_PWM,Buzzer_PWM}, USB{Data_-,Data_+,CC1,CC2}; removed JTAG{DO&SWO,NJTRST,MS&SWDIO,CLK,DI}
- sheet Sensors ports: added BMP{MOSI,MISO,SCK,NSS}, IMU{SCL,SDA,INTA,INTM}; removed none
Changed lines of the file:
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@@
 (kicad_sch (version 20230121) (generator eeschema)
   (paper "A4")
-  (bus (pts (xy 146.05 85.09) (xy 185.42 85.09))
+  (bus (pts (xy 200.025 80.01) (xy 213.36 80.01))
     (stroke (width 0) (type default))
   )
-  (sheet (at 185.42 64.77) (size 54.61 27.94) (fields_autoplaced)
+  (bus (pts (xy 106.045 84.455) (xy 145.415 84.455))
+    (stroke (width 0) (type default))
+  )
+  (bus (pts (xy 106.045 80.645) (xy 145.415 80.645))
+    (stroke (width 0) (type default))
+  )
+  (bus (pts (xy 106.045 72.39) (xy 145.415 72.39))
+    (stroke (width 0) (type default))
+  )
+  (bus (pts (xy 200.025 75.565) (xy 213.36 75.565))
+    (stroke (width 0) (type default))
+  )
+  (sheet (at 145.415 64.135) (size 54.61 27.94) (fields_autoplaced)
     (stroke (width 0.1524) (type solid))
     (fill (color 0 0 0 0.0000))
-    (property "Sheetname" "MCU" (at 185.42 64.0584 0)
+    (property "Sheetname" "MCU" (at 145.415 63.4234 0)
       (effects (font (size 1.27 1.27)) (justify left bottom))
     )
-    (property "Sheetfile" "MCU.kicad_sch" (at 185.42 93.2946 0)
+    (property "Sheetfile" "MCU.kicad_sch" (at 145.415 92.6596 0)
       (effects (font (size 1.27 1.27)) (justify left top))
     )
-    (pin "JTAG{DO&SWO,NJTRST,MS&SWDIO,CLK,DI}" bidirectional (at 185.42 85.09 180)
+    (pin "BMP{MOSI,MISO,SCK,NSS}" bidirectional (at 200.025 75.565 0)
+      (effects (font (size 1.27 1.27)) (justify right))
+    )
+    (pin "USB{Data_-,Data_+,CC1,CC2}" bidirectional (at 145.415 80.645 180)
+      (effects (font (size 1.27 1.27)) (justify left))
+    )
+    (pin "IMU{SCL,SDA,INTA,INTM}" bidirectional (at 200.025 80.01 0)
+      (effects (font (size 1.27 1.27)) (justify right))
+    )
+    (pin "JTAG{DOSWO,NJTRST,MSSWDIO,CLK,DI}" bidirectional (at 145.415 84.455 180)
+      (effects (font (size 1.27 1.27)) (justify left))
+    )
+    (pin "MISC{RECOVERY_LED_PWM,Buzzer_PWM}" input (at 145.415 72.39 180)
       (effects (font (size 1.27 1.27)) (justify left))
     )
@@
     )
   )
-  (sheet (at 88.9 64.77) (size 57.15 31.75) (fields_autoplaced)
+  (sheet (at 48.895 64.135) (size 57.15 31.75) (fields_autoplaced)
     (stroke (width 0.1524) (type solid))
     (fill (color 0 0 0 0.0000))
-    (property "Sheetname" "Connectors + Power" (at 88.9 64.0584 0)
+    (property "Sheetname" "Connectors + Power" (at 48.895 63.4234 0)
       (effects (font (size 1.27 1.27)) (justify left bottom))
     )
-    (property "Sheetfile" "Connectors.kicad_sch" (at 88.9 97.1046 0)
+    (property "Sheetfile" "Connectors.kicad_sch" (at 48.895 96.4696 0)
       (effects (font (size 1.27 1.27)) (justify left top))
     )
-    (pin "JTAG{DO&SWO,NJTRST,MS&SWDIO,CLK,DI}" bidirectional (at 146.05 85.09 0)
+    (pin "USB{Data_-,Data_+,CC1,CC2}" bidirectional (at 106.045 80.645 0)
+      (effects (font (size 1.27 1.27)) (justify right))
+    )
+    (pin "JTAG{DOSWO,NJTRST,MSSWDIO,CLK,DI}" bidirectional (at 106.045 84.455 0)
+      (effects (font (size 1.27 1.27)) (justify right))
+    )
+    (pin "MISC{RECOVERY_LED_PWM,Buzzer_PWM}" input (at 106.045 72.39 0)
       (effects (font (size 1.27 1.27)) (justify right))
     )
@@
     )
   )
-  (sheet (at 173.99 138.43) (size 46.99 16.51) (fields_autoplaced)
+  (sheet (at 213.36 69.85) (size 46.99 16.51) (fields_autoplaced)
     (stroke (width 0.1524) (type solid))
     (fill (color 0 0 0 0.0000))
-    (property "Sheetname" "Sensors" (at 173.99 137.7184 0)
+    (property "Sheetname" "Sensors" (at 213.36 69.1384 0)
       (effects (font (size 1.27 1.27)) (justify left bottom))
     )
-    (property "Sheetfile" "sensors.kicad_sch" (at 173.99 155.5246 0)
+    (property "Sheetfile" "sensors.kicad_sch" (at 213.36 86.9446 0)
       (effects (font (size 1.27 1.27)) (justify left top))
     )
+    (pin "BMP{MOSI,MISO,SCK,NSS}" bidirectional (at 213.36 75.565 180)
+      (effects (font (size 1.27 1.27)) (justify left))
+    )
+    (pin "IMU{SCL,SDA,INTA,INTM}" bidirectional (at 213.36 80.01 180)
+      (effects (font (size 1.27 1.27)) (justify left))
+    )
     (instances
