File: lil-flite/sensors.kicad_sch (KiCad schematic)
At the start: 2 parts, among them U102 BMP280, U302 MC6470

Commit message: Almost finished
Need to double check everything
routing done
more vias maybe
Parts:
- added C410 (x3): 100nF, Capacitor_SMD:C_0603_1608Metric_Pad1.08x0.95mm_HandSolder, symbol PCM_Generic-50:C,IEC
- added R401 (x3): 4k7, Resistor_SMD:R_0603_1608Metric_Pad0.98x0.95mm_HandSolder, symbol PCM_Generic-50:R,IEC
Connections:
- net GND: now reaches U102.1 (GND)
- net GND: now also U102.7 (GND), U302.1 (A5), U302.9 (GND), C410.1 (+), C410.1 (+), C410.1 (+)
- net BMP.NSS: now reaches U102.2 (CSB)
- net BMP.MOSI: now reaches U102.3 (SDI)
- net BMP.SCK: now reaches U102.4 (SCK)
- net BMP.MISO: now reaches U102.5 (SDO)
- net VCC: now reaches U102.6 (VDDIO)
- net VCC: now also U102.8 (VDD), U302.3 (VDDIO), U302.7 (VDDM), C410.2 (-), C410.2 (-), C410.2 (-), R401.2 (-), R401.2 (-), R401.2 (-)
- net IMU.SCL: now reaches U302.12 (SCL)
- net IMU.SCL: now also R401.1 (+)
- net IMU.SDA: now reaches U302.2 (SDA)
- net IMU.SDA: now also R401.1 (+)
- net IMU.INTA: now reaches U302.5 (INTA)
- net IMU.INTA: now also R401.1 (+)
- net IMU.INTM: now reaches U302.6 (INTM)
- no-connect marks 0 -> 3
Other:
- moved on the sheet: U102
